File: Simon Says Game v1.1.brd (EAGLE design)
At the start: 182.3 x 130.9 mm, 25 parts, among them U1 ARDUINO-UNO-R3-SHIELD, U3 LCD-16X2JHD-162A

Commit message: Changed files to reflect version 1.1
Parts:
- added R11: 1k, Tinkercad:RESAD1016W63L850D250B
- added RPOT1: 250k, Tinkercad:HA-06-SM065
- moved R9 12.7 mm to (164.7, 64.3)
- moved RPOT9 12.7 mm to (167.2, 74.5)
Connections:
- new net RPOT1_P$1: R11.2, RPOT1.1
- new net U1_A4: RPOT1.2, U1.A4
- net U1_5V: now also RPOT1.3
- net U1_GND: now also R11.1
